File: Projects/Slip_Sensor/Hardware/PAT9125_Breakout/PAT9125_Breakout.brd (EAGLE design)
At the start: 17.7 x 17.1 mm, 5 parts, among them X1 TSW-106-07-G-S

Commit message: finalized PAT9125 breakout board for ordering
Parts:
- moved C3 6.02 mm to (18.3, 13.6)
- moved C1 3.00 mm to (18.3, 9.02)
- moved C2 3.00 mm to (18.3, 11.6)
- moved U$1 2.22 mm to (11.3, 9.53)
Routing:
- net 3V3: track 17.5 -> 15.1 mm
- net ID_SEL: track 7.78 -> 5.41 mm
- net MOTION: track 7.05 -> 4.69 mm
- net VDDA: track 3.99 -> 5.73 mm
- net SDA: track 6.41 -> 4.98 mm
- net SCL: track 7.13 -> 5.70 mm
Other:
- board size 17.7 x 17.1 mm -> 17.7 x 12.4 mm
- board text added: "ID"
- board text added: "MOT"
- board text added: "PAT9125 Breakout Chris Le"
- board text removed: "ID_SEL"
- board text removed: "MOTION"
- board text removed: "PAT9125 - CHrisLe"
