File: Projects/Slip_Sensor/Hardware/PAT9125_Breakout/PAT9125_Breakout.sch (EAGLE design)
At the start: 4 parts

Commit message: The changes I made to the PAT9125 breakout board.
Parts:
- added X1: TSW-106-07-G-S, con-samtec:TSW-106-07-G-S
- C1, C3: device rcl:C-EUC0402 -> rcl:C-EUC0603
Connections:
- net 3V3: now also X1-5.1
- net GND: now also X1-6.1
- net ID_SEL: now also X1-4.1
- net MOTION: now also X1-3.1
- net SCL: now also X1-1.1
- net SDA: now also X1-2.1
Changed lines of the file:
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@@
 </variantdefs>
 <classes>
-<class number="0" name="default" width="0" drill="0">
+<class number="0" name="default" width="0.3048" drill="0.508">
+<clearance class="0" value="0.254"/>
 </class>
 </classes>
 <parts>
 <part name="U$1" library="Limbo" deviceset="PAT9125EL" device=""/>
-<part name="C1" library="rcl" library_urn="urn:adsk.eagle:library:334" deviceset="C-EU" device="C0402" package3d_urn="urn:adsk.eagle:package:23626/2" value="10uF"/>
+<part name="C1" library="rcl" library_urn="urn:adsk.eagle:library:334" deviceset="C-EU" device="C0603" package3d_urn="urn:adsk.eagle:package:23616/2" value="10uF"/>
 <part name="C2" library="rcl" library_urn="urn:adsk.eagle:library:334" deviceset="C-EU" device="C0603" package3d_urn="urn:adsk.eagle:package:23616/2" value=".1uF"/>
-<part name="C3" library="rcl" library_urn="urn:adsk.eagle:library:334" deviceset="C-EU" device="C0402" package3d_urn="urn:adsk.eagle:package:23626/2" value="4.7uF"/>
+<part name="C3" library="rcl" library_urn="urn:adsk.eagle:library:334" deviceset="C-EU" device="C0603" package3d_urn="urn:adsk.eagle:package:23616/2" value="4.7uF"/>
+<part name="X1" library="con-samtec" library_urn="urn:adsk.eagle:library:184" deviceset="TSW-106-*-G-S" device="" technology="07"/>
 </parts>
 <sheets>
@@
 <attribute name="NAME" x="24.384" y="48.641" size="1.778" layer="95"/>
 <attribute name="VALUE" x="24.384" y="43.561" size="1.778" layer="96"/>
+</instance>
+<instance part="X1" gate="-1" x="34.29" y="78.74" smashed="yes">
+<attribute name="VALUE" x="33.02" y="80.01" size="1.778" layer="96"/>
+<attribute name="NAME" x="36.83" y="77.978" size="1.524" layer="95"/>
+</instance>
+<instance part="X1" gate="-2" x="34.29" y="76.2" smashed="yes">
+<attribute name="NAME" x="36.83" y="75.438" size="1.524" layer="95"/>
+</instance>
+<instance part="X1" gate="-3" x="34.29" y="73.66" smashed="yes">
+<attribute name="NAME" x="36.83" y="72.898" size="1.524" layer="95"/>
+</instance>
+<instance part="X1" gate="-4" x="34.29" y="71.12" smashed="yes">
+<attribute name="NAME" x="36.83" y="70.358" size="1.524" layer="95"/>
+</instance>
+<instance part="X1" gate="-5" x="34.29" y="68.58" smashed="yes">
+<attribute name="NAME" x="36.83" y="67.818" size="1.524" layer="95"/>
+</instance>
+<instance part="X1" gate="-6" x="34.29" y="66.04" smashed="yes">
+<attribute name="NAME" x="36.83" y="65.278" size="1.524" layer="95"/>
 </instance>
 </instances>
@@
 <label x="-2.54" y="53.34" size="1.778" layer="95" rot="R90" xref="yes"/>
 </segment>
+<segment>
+<pinref part="X1" gate="-5" pin="1"/>
+<wire x1="30.48" y1="68.58" x2="31.75" y2="68.58" width="0.1524" layer="91"/>
+<label x="25.4" y="68.58" size="1.778" layer="95"/>
+</segment>
 </net>
 <net name="GND" class="0">
@@
 <wire x1="22.86" y1="40.64" x2="22.86" y2="43.18" width="0.1524" layer="91"/>
 <pinref part="C2" gate="G$1" pin="2"/>
-<wire x1="10.16" y1="43.18" x2="10.16" y2="40.64" width="0.1524" layer="91"/>
-<wire x1="22.86" y1="40.64" x2="10.16" y2="40.64" width="0.1524" layer="91"/>
-<wire x1="10.16" y1="40.64" x2="-2.54" y2="40.64" width="0.1524" layer="91"/>
-<junction x="10.16" y="40.64"/>
-<wire x1="10.16" y1="40.64" x2="10.16" y2="38.1" width="0.1524" layer="91"/>
-<label x="10.16" y="38.1" size="1.778" layer="95" rot="R270" xref="yes"/>
+<wire x1="10.16" y1="43.18" x2="10.16" y2="38.1" width="0.1524" layer="91"/>
+<wire x1="22.86" y1="40.64" x2="10.16" y2="38.1" width="0.1524" layer="91"/>
+<wire x1="10.16" y1="38.1" x2="-2.54" y2="40.64" width="0.1524" layer="91"/>
+<junction x="10.16" y="38.1"/>
+<wire x1="10.16" y1="38.1" x2="10.16" y2="35.56" width="0.1524" layer="91"/>
+<label x="10.16" y="35.56" size="1.778" layer="95" rot="R270" xref="yes"/>
 </segment>
 <segment>
@@
 <wire x1="50.8" y1="38.1" x2="40.64" y2="38.1" width="0.1524" layer="91"/>
 <label x="40.64" y="38.1" size="1.778" layer="95"/>
+</segment>
+<segment>
+<pinref part="X1" gate="-6" pin="1"/>
+<wire x1="30.48" y1="66.04" x2="31.75" y2="66.04" width="0.1524" layer="91"/>
+<label x="25.4" y="66.04" size="1.778" layer="95"/>
 </segment>
 </net>
@@
 <label x="86.36" y="53.34" size="1.778" layer="95" rot="MR0"/>
 </segment>
+<segment>
+<pinref part="X1" gate="-4" pin="1"/>
+<wire x1="30.48" y1="71.12" x2="31.75" y2="71.12" width="0.1524" layer="91"/>
+<label x="25.4" y="71.12" size="1.778" layer="95"/>
+</segment>
 </net>
 <net name="MOTION" class="0">
@@
 <wire x1="76.2" y1="48.26" x2="86.36" y2="48.26" width="0.1524" layer="91"/>
 <label x="86.36" y="48.26" size="1.778" layer="95" rot="MR0"/>
+</segment>
+<segment>
+<pinref part="X1" gate="-3" pin="1"/>
+<wire x1="30.48" y1="73.66" x2="31.75" y2="73.66" width="0.1524" layer="91"/>
+<label x="25.4" y="73.66" size="1.778" layer="95"/>
 </segment>
 </net>
@@
 <label x="86.36" y="43.18" size="1.778" layer="95" rot="MR0"/>
 </segment>
+<segment>
+<pinref part="X1" gate="-2" pin="1"/>
+<wire x1="31.75" y1="76.2" x2="30.48" y2="76.2" width="0.1524" layer="91"/>
+<label x="25.4" y="76.2" size="1.778" layer="95"/>
+</segment>
 </net>
 <net name="SCL" class="0">
@@
 <label x="86.36" y="38.1" size="1.778" layer="95" rot="MR0"/>
 </segment>
+<segment>
+<pinref part="X1" gate="-1" pin="1"/>
+<wire x1="30.48" y1="78.74" x2="31.75" y2="78.74" width="0.1524" layer="91"/>
+<label x="25.4" y="78.74" size="1.778" layer="95"/>
+</segment>
 </net>
