File: Projects/Palm_Hub/palmhub_kicad_v2/palm hub v2 021424.kicad_sch (KiCad schematic)
At the start: 27 parts, among them J1 Conn_01x08_Male, U1 adc108s, U2 Pico, U3 LP2950-3.0_TO92

Commit message: new schematic upload
Connections:
- net at U1.1 (CS): now also U2.7 (GPIO5); no longer U2.6 (GPIO4)
- net at U1.15 (DOUT): now also U2.6 (GPIO4); no longer U2.9 (GPIO6)
- net at U1.16 (SCLK): now also U2.9 (GPIO6); no longer U2.7 (GPIO5)
Changed lines of the file:
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@@
-    (stroke (width 0) (type default))
-  )
-  (wire (pts (xy 123.19 109.22) (xy 107.95 109.22))
     (stroke (width 0) (type default))
   )
   (wire (pts (xy 115.57 111.76) (xy 123.19 111.76))
+    (stroke (width 0) (type default))
+  )
+  (wire (pts (xy 113.03 62.23) (xy 106.68 62.23))
     (stroke (width 0) (type default))
   )
@@
   )
   (wire (pts (xy 115.57 130.81) (xy 130.81 130.81))
-    (stroke (width 0) (type default))
-  )
-  (wire (pts (xy 107.95 59.69) (xy 113.03 59.69))
     (stroke (width 0) (type default))
   )
@@
     (stroke (width 0) (type default))
   )
-  (wire (pts (xy 140.97 111.76) (xy 139.7 111.76))
+  (wire (pts (xy 139.7 111.76) (xy 146.05 111.76))
+    (stroke (width 0) (type default))
+  )
+  (wire (pts (xy 101.6 59.69) (xy 101.6 104.14))
     (stroke (width 0) (type default))
   )
@@
     (stroke (width 0) (type default))
   )
-  (wire (pts (xy 139.7 106.68) (xy 139.7 109.22))
+  (wire (pts (xy 130.81 130.81) (xy 130.81 132.08))
     (stroke (width 0) (type default))
   )
-  (wire (pts (xy 109.22 106.68) (xy 139.7 106.68))
-    (stroke (width 0) (type default))
-  )
-  (wire (pts (xy 130.81 130.81) (xy 130.81 132.08))
+  (wire (pts (xy 109.22 106.68) (xy 109.22 67.31))
     (stroke (width 0) (type default))
   )
@@
     (stroke (width 0) (type default))
   )
-  (wire (pts (xy 142.24 104.14) (xy 142.24 114.3))
-    (stroke (width 0) (type default))
-  )
-  (wire (pts (xy 110.49 105.41) (xy 140.97 105.41))
+  (wire (pts (xy 139.7 109.22) (xy 142.24 109.22))
     (stroke (width 0) (type default))
   )
@@
     (stroke (width 0) (type default))
   )
-  (wire (pts (xy 110.49 67.31) (xy 110.49 105.41))
-    (stroke (width 0) (type default))
-  )
   (wire (pts (xy 46.99 149.86) (xy 44.45 149.86))
     (stroke (width 0) (type default))
   )
-  (wire (pts (xy 109.22 62.23) (xy 109.22 106.68))
+  (wire (pts (xy 106.68 62.23) (xy 106.68 109.22))
     (stroke (width 0) (type default))
   )
@@
     (stroke (width 0) (type default))
   )
+  (wire (pts (xy 109.22 67.31) (xy 113.03 67.31))
+    (stroke (width 0) (type default))
+  )
   (wire (pts (xy 45.72 166.37) (xy 43.18 166.37))
     (stroke (width 0) (type default))
   )
-  (wire (pts (xy 111.76 69.85) (xy 111.76 104.14))
+  (wire (pts (xy 111.76 69.85) (xy 111.76 101.6))
     (stroke (width 0) (type default))
   )
@@
     (stroke (width 0) (type default))
   )
-  (wire (pts (xy 142.24 114.3) (xy 139.7 114.3))
+  (wire (pts (xy 113.03 59.69) (xy 101.6 59.69))
+    (stroke (width 0) (type default))
+  )
+  (wire (pts (xy 139.7 114.3) (xy 148.59 114.3))
     (stroke (width 0) (type default))
   )
@@
     (stroke (width 0) (type default))
   )
-  (wire (pts (xy 140.97 105.41) (xy 140.97 111.76))
+  (wire (pts (xy 142.24 109.22) (xy 142.24 106.68))
     (stroke (width 0) (type default))
   )
-  (wire (pts (xy 113.03 62.23) (xy 109.22 62.23))
+  (wire (pts (xy 146.05 111.76) (xy 146.05 104.14))
     (stroke (width 0) (type default))
   )
@@
     (stroke (width 0) (type default))
   )
-  (wire (pts (xy 107.95 109.22) (xy 107.95 59.69))
+  (wire (pts (xy 106.68 109.22) (xy 123.19 109.22))
     (stroke (width 0) (type default))
   )
-  (wire (pts (xy 113.03 67.31) (xy 110.49 67.31))
-    (stroke (width 0) (type default))
-  )
-  (wire (pts (xy 111.76 104.14) (xy 142.24 104.14))
+  (wire (pts (xy 148.59 114.3) (xy 148.59 101.6))
     (stroke (width 0) (type default))
   )
   (wire (pts (xy 80.645 116.84) (xy 75.565 116.84))
+    (stroke (width 0) (type default))
+  )
+  (wire (pts (xy 142.24 106.68) (xy 109.22 106.68))
+    (stroke (width 0) (type default))
+  )
+  (wire (pts (xy 146.05 104.14) (xy 101.6 104.14))
     (stroke (width 0) (type default))
   )
@@
     (stroke (width 0) (type default))
   )
+  (wire (pts (xy 148.59 101.6) (xy 111.76 101.6))
+    (stroke (width 0) (type default))
+  )
